File: pcb/tes1.brd (EAGLE design)
At the start: 7 x 6.9 mm, 33 parts, among them IC1 STM32F10XCXT6, Q1 BC817-40SMD, Q2 BC817-40SMD, Q3 BC817-40SMD, Q4 8mhz

Commit message: Pengujian tahap 1
Parts:
- RVA: value (none) -> 4k7
- RVB: value (none) -> 1k5
Connections:
- removed net N$8: S1.3
- net VSS: now also S1.3
Changed lines of the file:
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@@
 <attribute name="OC_FARNELL" value="unknown" x="37.465" y="13.716" size="1.778" layer="27" rot="R270" display="off"/>
 </element>
-<element name="RVA" library="resistor" package="R0805" value="" x="51.689" y="70.485" rot="MR180"/>
-<element name="RVB" library="resistor" package="R0805" value="" x="51.689" y="68.199" rot="MR180"/>
+<element name="RVA" library="resistor" package="R0805" value="4k7" x="51.689" y="70.485" rot="MR180"/>
+<element name="RVB" library="resistor" package="R0805" value="1k5" x="51.689" y="68.199" rot="MR180"/>
 <element name="CV" library="resistor" package="C0805" value="100n" x="51.689" y="65.786" rot="MR0"/>
 <element name="PV" library="con-jack" package="SPC4077" value="" x="47.879" y="33.274" rot="R90">
@@
 <wire x1="41.148" y1="76.835" x2="41.021" y2="76.962" width="0.6096" layer="16"/>
 <wire x1="41.021" y1="76.962" x2="27.94" y2="76.962" width="0.6096" layer="16"/>
+<contactref element="S1" pad="3"/>
+<wire x1="40.695" y1="58.686" x2="45.1358" y2="58.6994" width="0" layer="19" extent="16-16"/>
 </signal>
 <signal name="V2">
@@
 <wire x1="26.924" y1="59.563" x2="26.797" y2="59.69" width="0.6096" layer="16"/>
 </signal>
-<signal name="N$8">
-<contactref element="S1" pad="3"/>
-</signal>
 <signal name="SW">
