File: pcb/tes1.sch (EAGLE design)
At the start: 33 parts, among them IC1 STM32F10XCXT6, Q1 BC817-40SMD, Q2 BC817-40SMD, Q3 BC817-40SMD, Q4 8mhz

Commit message: Pengujian tahap 1
Parts:
- RVA: value (none) -> 4k7
- RVB: value (none) -> 1k5
Connections:
- removed net N$8: S1.P
- net VSS: now also S1.P
Changed lines of the file:
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@@
 <part name="BATT3" library="con-ptr500" deviceset="AK300/2" device=""/>
 <part name="BATT4" library="con-ptr500" deviceset="AK300/2" device=""/>
-<part name="RVA" library="resistor" deviceset="R-EU_" device="R0805"/>
-<part name="RVB" library="resistor" deviceset="R-EU_" device="R0805"/>
+<part name="RVA" library="resistor" deviceset="R-EU_" device="R0805" value="4k7"/>
+<part name="RVB" library="resistor" deviceset="R-EU_" device="R0805" value="1k5"/>
 <part name="CV" library="resistor" deviceset="C-EU" device="C0805" value="100n"/>
 <part name="PV" library="con-jack" deviceset="JACK-PLUG" device="0"/>
@@
 <label x="129.54" y="5.08" size="1.778" layer="95"/>
 </segment>
+<segment>
+<pinref part="S1" gate="1" pin="P"/>
+<wire x1="-7.62" y1="35.56" x2="-10.16" y2="35.56" width="0.1524" layer="91"/>
+<label x="-10.16" y="35.56" size="1.778" layer="95" rot="R180"/>
+</segment>
 </net>
 <net name="V2" class="0">
@@
 </segment>
 </net>
-<net name="N$8" class="0">
-<segment>
-<pinref part="S1" gate="1" pin="P"/>
-<wire x1="-7.62" y1="35.56" x2="-10.16" y2="35.56" width="0.1524" layer="91"/>
-<label x="-10.16" y="35.56" size="1.778" layer="95" rot="R180"/>
-</segment>
-</net>
