File: test-bench/led-056/led-056.sch (KiCad schematic (older format))
At the start: 15 parts, among them IC1 4511D, P1 CONN_02X05, U1 PC817, U2 PC817, U3 PC817

Commit message: BOM
Parts:
- AFF1, AFF2, AFF3: footprint Displays_7-Segment:7SegmentLED_SBC18-11EGWA -> Displays_7-Segment:7SegmentLED_LTS6760_LTS6780
- P1: footprint Pin_Headers:Pin_Header_Angled_2x05 -> Pin_Headers:Pin_Header_Straight_2x05
Changed lines of the file:
@@
 F 0 "P1" H 2800 3000 50  0000 C CNN
 F 1 "CONN_02X05" H 2800 2400 50  0000 C CNN
-F 2 "Pin_Headers:Pin_Header_Angled_2x05" H 2800 1500 60  0001 C CNN
+F 2 "Pin_Headers:Pin_Header_Straight_2x05" H 2800 1500 60  0001 C CNN
 F 3 "" H 2800 1500 60  0000 C CNN
 	1    2800 2700
@@
 F 0 "AFF1" H 7400 3450 60  0000 C CNN
 F 1 "7SEGMENTS" H 7400 2450 60  0000 C CNN
-F 2 "Displays_7-Segment:7SegmentLED_SBC18-11EGWA" H 7400 2900 60  0001 C CNN
+F 2 "Displays_7-Segment:7SegmentLED_LTS6760_LTS6780" H 7400 2900 60  0001 C CNN
 F 3 "" H 7400 2900 60  0000 C CNN
 	1    7400 2900
@@
 F 0 "AFF2" H 7400 4500 60  0000 C CNN
 F 1 "7SEGMENTS" H 7400 3500 60  0000 C CNN
-F 2 "Displays_7-Segment:7SegmentLED_SBC18-11EGWA" H 7400 3950 60  0001 C CNN
+F 2 "Displays_7-Segment:7SegmentLED_LTS6760_LTS6780" H 7400 3950 60  0001 C CNN
 F 3 "" H 7400 3950 60  0000 C CNN
 	1    7400 3950
@@
 F 0 "AFF3" H 7400 5550 60  0000 C CNN
 F 1 "7SEGMENTS" H 7400 4550 60  0000 C CNN
-F 2 "Displays_7-Segment:7SegmentLED_SBC18-11EGWA" H 7400 5000 60  0001 C CNN
+F 2 "Displays_7-Segment:7SegmentLED_LTS6760_LTS6780" H 7400 5000 60  0001 C CNN
 F 3 "" H 7400 5000 60  0000 C CNN
 	1    7400 5000
