File: test-bench/led-100/led-100.sch (KiCad schematic (older format))
At the start: 17 parts, among them IC1 4511D, P1 CONN_02X05, U1 PC817, U2 PC817, U3 PC817, U4 PC817

Commit message: BOM
Parts:
- P1: footprint Resistors_ThroughHole:Resistor_Horizontal_RM10mm -> Pin_Headers:Pin_Header_Straight_2x05
Changed lines of the file:
@@
 F 0 "P1" H 2650 2350 50  0000 C CNN
 F 1 "CONN_02X05" H 2650 1750 50  0000 C CNN
-F 2 "Resistors_ThroughHole:Resistor_Horizontal_RM10mm" H 2650 850 60  0001 C CNN
+F 2 "Pin_Headers:Pin_Header_Straight_2x05" H 2650 850 60  0001 C CNN
 F 3 "" H 2650 850 60  0000 C CNN
 	1    2650 2050
