File: test-bench/mainboard/mainboard.kicad_pcb (KiCad board)
At the start: 2 copper layers, 33 parts, among them CON1 BARREL_JACK, IC1 ATMEGA128-A, IC2 LM2596S, U1 PCF8563, Y1 Crystal_Small

Commit message: BOM
Parts:
- IC1: footprint Housings_QFP:TQFP-64_14x14mm_Pitch0.8mm -> Housings_QFP:LQFP-64_14x14mm_Pitch0.8mm
- moved IC1 0.29 mm to (153.7, 100.0)
