File: test-bench/mainboard/mainboard.sch (KiCad schematic (older format))
At the start: 33 parts, among them CON1 BARREL_JACK, IC1 ATMEGA128-A, IC2 LM2596S, U1 PCF8563, Y1 Crystal_Small

Commit message: BOM
Parts:
- IC1: footprint Housings_QFP:TQFP-64_14x14mm_Pitch0.8mm -> Housings_QFP:LQFP-64_14x14mm_Pitch0.8mm
Changed lines of the file:
@@
 F 0 "IC1" H 4000 4900 40  0000 L BNN
 F 1 "ATMEGA128-A" H 5900 1050 40  0000 L BNN
-F 2 "Housings_QFP:TQFP-64_14x14mm_Pitch0.8mm" H 5150 3000 30  0001 C CIN
+F 2 "Housings_QFP:LQFP-64_14x14mm_Pitch0.8mm" H 5150 3000 30  0001 C CIN
 F 3 "" H 5150 3000 60  0000 C CNN
 	1    5150 3000
@@
 $EndComp
 $Comp
-L VCC #PWR011
+L VCC #PWR09
 U 1 1 564D564F
 P 3050 3050
-F 0 "#PWR011" H 3050 2900 50  0001 C CNN
+F 0 "#PWR09" H 3050 2900 50  0001 C CNN
 F 1 "VCC" H 3050 3200 50  0000 C CNN
 F 2 "" H 3050 3050 60  0000 C CNN
@@
 $EndComp
 $Comp
-L GND #PWR012
+L GND #PWR010
 U 1 1 564D5655
 P 3300 3050
-F 0 "#PWR012" H 3300 2800 50  0001 C CNN
+F 0 "#PWR010" H 3300 2800 50  0001 C CNN
 F 1 "GND" H 3300 2900 50  0000 C CNN
 F 2 "" H 3300 3050 60  0000 C CNN
@@
 $EndComp
 $Comp
-L GND #PWR013
+L GND #PWR011
 U 1 1 564D725B
 P 7950 1950
-F 0 "#PWR013" H 7950 1700 50  0001 C CNN
+F 0 "#PWR011" H 7950 1700 50  0001 C CNN
 F 1 "GND" H 7950 1800 50  0000 C CNN
 F 2 "" H 7950 1950 60  0000 C CNN
@@
 $EndComp
 $Comp
-L VCC #PWR014
+L VCC #PWR012
 U 1 1 564D81F8
 P 9000 900
-F 0 "#PWR014" H 9000 750 50  0001 C CNN
+F 0 "#PWR012" H 9000 750 50  0001 C CNN
 F 1 "VCC" H 9000 1050 50  0000 C CNN
 F 2 "" H 9000 900 60  0000 C CNN
@@
 $EndComp
 $Comp
-L VCC #PWR015
+L VCC #PWR013
 U 1 1 564DB2DE
 P 7600 2450
-F 0 "#PWR015" H 7600 2300 50  0001 C CNN
+F 0 "#PWR013" H 7600 2300 50  0001 C CNN
 F 1 "VCC" H 7600 2600 50  0000 C CNN
 F 2 "" H 7600 2450 60  0000 C CNN
@@
 $EndComp
 $Comp
-L GND #PWR016
+L GND #PWR014
 U 1 1 564DB5BF
 P 8300 2850
-F 0 "#PWR016" H 8300 2600 50  0001 C CNN
+F 0 "#PWR014" H 8300 2600 50  0001 C CNN
 F 1 "GND" H 8300 2700 50  0000 C CNN
 F 2 "" H 8300 2850 60  0000 C CNN
@@
 $EndComp
 $Comp
-L VCC #PWR017
+L VCC #PWR015
 U 1 1 564DC3C5
 P 8800 2450
-F 0 "#PWR017" H 8800 2300 50  0001 C CNN
+F 0 "#PWR015" H 8800 2300 50  0001 C CNN
 F 1 "VCC" H 8800 2600 50  0000 C CNN
 F 2 "" H 8800 2450 60  0000 C CNN
@@
 $EndComp
 $Comp
-L GND #PWR018
+L GND #PWR016
 U 1 1 564DC3CC
 P 9500 2850
-F 0 "#PWR018" H 9500 2600 50  0001 C CNN
+F 0 "#PWR016" H 9500 2600 50  0001 C CNN
 F 1 "GND" H 9500 2700 50  0000 C CNN
 F 2 "" H 9500 2850 60  0000 C CNN
@@
 $EndComp
 $Comp
-L VCC #PWR019
+L VCC #PWR017
 U 1 1 564DC70B
 P 7650 3200
-F 0 "#PWR019" H 7650 3050 50  0001 C CNN
+F 0 "#PWR017" H 7650 3050 50  0001 C CNN
 F 1 "VCC" H 7650 3350 50  0000 C CNN
 F 2 "" H 7650 3200 60  0000 C CNN
@@
 $EndComp
 $Comp
-L GND #PWR020
+L GND #PWR018
 U 1 1 564DC712
 P 8350 3600
-F 0 "#PWR020" H 8350 3350 50  0001 C CNN
+F 0 "#PWR018" H 8350 3350 50  0001 C CNN
 F 1 "GND" H 8350 3450 50  0000 C CNN
 F 2 "" H 8350 3600 60  0000 C CNN
@@
 $EndComp
 $Comp
-L VCC #PWR021
+L VCC #PWR019
 U 1 1 564DC72B
 P 8850 3200
-F 0 "#PWR021" H 8850 3050 50  0001 C CNN
+F 0 "#PWR019" H 8850 3050 50  0001 C CNN
 F 1 "VCC" H 8850 3350 50  0000 C CNN
 F 2 "" H 8850 3200 60  0000 C CNN
@@
 $EndComp
 $Comp
-L GND #PWR022
+L GND #PWR020
 U 1 1 564DC732
 P 9550 3600
-F 0 "#PWR022" H 9550 3350 50  0001 C CNN
+F 0 "#PWR020" H 9550 3350 50  0001 C CNN
 F 1 "GND" H 9550 3450 50  0000 C CNN
 F 2 "" H 9550 3600 60  0000 C CNN
@@
 $EndComp
 $Comp
-L VCC #PWR023
+L VCC #PWR021
 U 1 1 564DCD33
 P 7650 4000
-F 0 "#PWR023" H 7650 3850 50  0001 C CNN
+F 0 "#PWR021" H 7650 3850 50  0001 C CNN
 F 1 "VCC" H 7650 4150 50  0000 C CNN
 F 2 "" H 7650 4000 60  0000 C CNN
@@
 $EndComp
 $Comp
-L GND #PWR024
+L GND #PWR022
 U 1 1 564DCD3A
 P 8350 4400
-F 0 "#PWR024" H 8350 4150 50  0001 C CNN
+F 0 "#PWR022" H 8350 4150 50  0001 C CNN
 F 1 "GND" H 8350 4250 50  0000 C CNN
 F 2 "" H 8350 4400 60  0000 C CNN
@@
 $EndComp
 $Comp
-L VCC #PWR025
+L VCC #PWR023
 U 1 1 564DCD53
 P 8850 4000
-F 0 "#PWR025" H 8850 3850 50  0001 C CNN
+F 0 "#PWR023" H 8850 3850 50  0001 C CNN
 F 1 "VCC" H 8850 4150 50  0000 C CNN
 F 2 "" H 8850 4000 60  0000 C CNN
@@
 $EndComp
 $Comp
-L GND #PWR026
+L GND #PWR024
 U 1 1 564DCD5A
 P 9550 4400
-F 0 "#PWR026" H 9550 4150 50  0001 C CNN
+F 0 "#PWR024" H 9550 4150 50  0001 C CNN
 F 1 "GND" H 9550 4250 50  0000 C CNN
 F 2 "" H 9550 4400 60  0000 C CNN
@@
 $EndComp
 $Comp
-L VCC #PWR027
+L VCC #PWR025
 U 1 1 564DCD73
 P 7700 4750
-F 0 "#PWR027" H 7700 4600 50  0001 C CNN
+F 0 "#PWR025" H 7700 4600 50  0001 C CNN
 F 1 "VCC" H 7700 4900 50  0000 C CNN
 F 2 "" H 7700 4750 60  0000 C CNN
@@
 $EndComp
 $Comp
-L GND #PWR028
+L GND #PWR026
 U 1 1 564DCD7A
 P 8400 5150
-F 0 "#PWR028" H 8400 4900 50  0001 C CNN
+F 0 "#PWR026" H 8400 4900 50  0001 C CNN
 F 1 "GND" H 8400 5000 50  0000 C CNN
 F 2 "" H 8400 5150 60  0000 C CNN
@@
 $EndComp
 $Comp
-L VCC #PWR029
+L VCC #PWR027
 U 1 1 564DCD93
 P 8900 4750
-F 0 "#PWR029" H 8900 4600 50  0001 C CNN
+F 0 "#PWR027" H 8900 4600 50  0001 C CNN
 F 1 "VCC" H 8900 4900 50  0000 C CNN
 F 2 "" H 8900 4750 60  0000 C CNN
@@
 $EndComp
 $Comp
-L GND #PWR030
+L GND #PWR028
 U 1 1 564DCD9A
 P 9600 5150
-F 0 "#PWR030" H 9600 4900 50  0001 C CNN
+F 0 "#PWR028" H 9600 4900 50  0001 C CNN
 F 1 "GND" H 9600 5000 50  0000 C CNN
 F 2 "" H 9600 5150 60  0000 C CNN
@@
 $EndComp
 $Comp
-L GND #PWR032
+L GND #PWR029
 U 1 1 564E1C67
 P 2850 4350
-F 0 "#PWR032" H 2850 4100 50  0001 C CNN
+F 0 "#PWR029" H 2850 4100 50  0001 C CNN
 F 1 "GND" H 2850 4200 50  0000 C CNN
 F 2 "" H 2850 4350 60  0000 C CNN
@@
 $EndComp
 $Comp
-L GND #PWR033
+L GND #PWR030
 U 1 1 564D58E1
 P 4450 5600
-F 0 "#PWR033" H 4450 5350 50  0001 C CNN
+F 0 "#PWR030" H 4450 5350 50  0001 C CNN
 F 1 "GND" H 4450 5450 50  0000 C CNN
 F 2 "" H 4450 5600 60  0000 C CNN
@@
 Connection ~ 5350 5950
 $Comp
-L VCC #PWR034
+L VCC #PWR031
 U 1 1 564D8F12
 P 7000 5400
-F 0 "#PWR034" H 7000 5250 50  0001 C CNN
+F 0 "#PWR031" H 7000 5250 50  0001 C CNN
 F 1 "VCC" H 7000 5550 50  0000 C CNN
 F 2 "" H 7000 5400 60  0000 C CNN
@@
 	7000 5850 7000 5400
 $Comp
-L VCC #PWR?
+L VCC #PWR032
 U 1 1 564D5A9B
 P 3300 3450
-F 0 "#PWR?" H 3300 3300 50  0001 C CNN
+F 0 "#PWR032" H 3300 3300 50  0001 C CNN
 F 1 "VCC" H 3300 3600 50  0000 C CNN
 F 2 "" H 3300 3450 60  0000 C CNN
