File: test-bench/date/date.kicad_pcb (KiCad board)
At the start: 2 copper layers, 90.7 x 44.9 mm, 13 parts, among them P1 CONN_02X08, U1 PC817, U2 PC817, U3 PC817, U4 PC817

Commit message: lapooor
Parts:
- added REF**: MountingHole_2-5mm, Mounting_Holes:MountingHole_2-5mm, F.Cu at (121.3, 119.0)
- added REF**: MountingHole_2-5mm, Mounting_Holes:MountingHole_2-5mm, F.Cu at (211.7, 80.0)
- added REF**: MountingHole_2-5mm, Mounting_Holes:MountingHole_2-5mm, F.Cu at (120.8, 80.1)
- added REF**: MountingHole_2-5mm, Mounting_Holes:MountingHole_2-5mm, F.Cu at (211.7, 119.1)
Other:
- board size 90.7 x 44.9 mm -> 97.6 x 46 mm
Changed lines of the file:
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@@
 (kicad_pcb (version 4) (host pcbnew "(2015-11-24 BZR 6329, Git e511afd)-product")
   (general
-    (links 52)
-    (no_connects 16)
-    (area 117.491667 80.783659 208.026221 120.32949)
+    (links 0)
+    (no_connects 0)
+    (area 112.314536 75.37488 220.383584 123.67418)
     (thickness 1.6)
     (drawings 4)
     (tracks 301)
     (zones 0)
-    (modules 13)
+    (modules 17)
     (nets 29)
   )
@@
   )
   (setup
-    (last_trace_width 0.5)
+    (last_trace_width 0.25)
     (user_trace_width 0.5)
     (user_trace_width 0.7)
@@
     )
   )
-  (gr_line (start 119 122.2) (end 118.8 77.7) (layer Edge.Cuts) (width 0.1))
-  (gr_line (start 209.5 122.4) (end 119 122.2) (layer Edge.Cuts) (width 0.1))
-  (gr_line (start 209.5 77.5) (end 209.5 122.4) (layer Edge.Cuts) (width 0.1))
-  (gr_line (start 118.8 77.7) (end 209.5 77.5) (layer Edge.Cuts) (width 0.1))
+  (module Mounting_Holes:MountingHole_2-5mm (layer F.Cu)
+    (at 121.3 119)
+    (descr "Mounting hole, Befestigungsbohrung, 2,5mm, No Annular, Kein Restring,")
+    (tags "Mounting hole, Befestigungsbohrung, 2,5mm, No Annular, Kein Restring,")
+    (fp_text reference REF** (at 0 -3.50012) (layer F.SilkS)
+      (effects (font (size 1 1) (thickness 0.15)))
+    )
+    (fp_text value MountingHole_2-5mm (at 0.09906 3.59918) (layer F.Fab)
+      (effects (font (size 1 1) (thickness 0.15)))
+    )
+    (fp_circle (center 0 0) (end 2.5 0) (layer Cmts.User) (width 0.381))
+    (pad 1 thru_hole circle (at 0 0) (size 2.5 2.5) (drill 2.5) (layers))
+  )
+  (module Mounting_Holes:MountingHole_2-5mm (layer F.Cu)
+    (at 211.7 80)
+    (descr "Mounting hole, Befestigungsbohrung, 2,5mm, No Annular, Kein Restring,")
+    (tags "Mounting hole, Befestigungsbohrung, 2,5mm, No Annular, Kein Restring,")
+    (fp_text reference REF** (at 0 -3.50012) (layer F.SilkS)
+      (effects (font (size 1 1) (thickness 0.15)))
+    )
+    (fp_text value MountingHole_2-5mm (at 0.09906 3.59918) (layer F.Fab)
+      (effects (font (size 1 1) (thickness 0.15)))
+    )
+    (fp_circle (center 0 0) (end 2.5 0) (layer Cmts.User) (width 0.381))
+    (pad 1 thru_hole circle (at 0 0) (size 2.5 2.5) (drill 2.5) (layers))
+  )
+  (module Mounting_Holes:MountingHole_2-5mm (layer F.Cu)
+    (at 120.8 80.1)
+    (descr "Mounting hole, Befestigungsbohrung, 2,5mm, No Annular, Kein Restring,")
+    (tags "Mounting hole, Befestigungsbohrung, 2,5mm, No Annular, Kein Restring,")
+    (fp_text reference REF** (at 0 -3.50012) (layer F.SilkS)
+      (effects (font (size 1 1) (thickness 0.15)))
+    )
+    (fp_text value MountingHole_2-5mm (at 0.09906 3.59918) (layer F.Fab)
+      (effects (font (size 1 1) (thickness 0.15)))
+    )
+    (fp_circle (center 0 0) (end 2.5 0) (layer Cmts.User) (width 0.381))
+    (pad 1 thru_hole circle (at 0 0) (size 2.5 2.5) (drill 2.5) (layers))
+  )
+  (module Mounting_Holes:MountingHole_2-5mm (layer F.Cu)
+    (at 211.7 119.1)
+    (descr "Mounting hole, Befestigungsbohrung, 2,5mm, No Annular, Kein Restring,")
+    (tags "Mounting hole, Befestigungsbohrung, 2,5mm, No Annular, Kein Restring,")
+    (fp_text reference REF** (at 0 -3.50012) (layer F.SilkS)
+      (effects (font (size 1 1) (thickness 0.15)))
+    )
+    (fp_text value MountingHole_2-5mm (at 0.09906 3.59918) (layer F.Fab)
+      (effects (font (size 1 1) (thickness 0.15)))
+    )
+    (fp_circle (center 0 0) (end 2.5 0) (layer Cmts.User) (width 0.381))
+    (pad 1 thru_hole circle (at 0 0) (size 2.5 2.5) (drill 2.5) (layers))
+  )
+  (gr_line (start 117.9 122.6) (end 117.8 76.6) (layer Edge.Cuts) (width 0.1))
+  (gr_line (start 215.4 122.6) (end 117.9 122.6) (layer Edge.Cuts) (width 0.1))
+  (gr_line (start 215.1 76.8) (end 215.4 122.6) (layer Edge.Cuts) (width 0.1))
+  (gr_line (start 117.8 76.6) (end 215.1 76.8) (layer Edge.Cuts) (width 0.1))
   (segment (start 129.301314 101.95) (end 134.25 101.95) (width 0.5) (layer F.Cu) (net 1))
   (segment (start 134.25 101.95) (end 137 99.2) (width 0.5) (layer F.Cu) (net 1))
@@
     (polygon
       (pts
-        (xy 118.8 77.7) (xy 209.5 77.5) (xy 209.5 122.4) (xy 119 122.2)
+        (xy 117.9 76.8) (xy 215.3 76.8) (xy 215.5 122.5) (xy 117.9 122.6)
       )
     )
@@
     (polygon
       (pts
-        (xy 118.8 77.7) (xy 209.5 77.5) (xy 209.5 122.4) (xy 119 122.2)
+        (xy 117.9 76.8) (xy 215.3 76.8) (xy 215.4 122.4) (xy 118.1 122.6)
       )
     )
