File: test-bench/value/value.kicad_pcb (KiCad board)
At the start: 2 copper layers, 59.4 x 37.3 mm, 10 parts, among them P1 CONN_02X08, U1 PC817, U2 PC817, U3 PC817

Commit message: design display beres
Routing:
- net /DA: track 94.6 -> 97.9 mm, vias 2 -> 1
- net /DB: track 57.7 -> 59.2 mm, vias 2 -> 1
- net /DC: track 37.5 -> 38.5 mm, vias 2 -> 1
- net GND: track 113.0 -> 113.6 mm, vias 0 -> 1
- net /LF: track 52.1 -> 52.6 mm, vias 3 -> 4
- net VCC: track 50.0 -> 50.5 mm, vias 0 -> 1
- net /LA: vias 4 -> 3
- net /LC: vias 4 -> 3
- net /LB: vias 4 -> 3

Commit message: lapooor
Parts:
- added REF**: MountingHole_2-5mm, Mounting_Holes:MountingHole_2-5mm, F.Cu at (219.4, 89.5)
- added REF**: MountingHole_2-5mm, Mounting_Holes:MountingHole_2-5mm, F.Cu at (219.3, 125.0)
- added REF**: MountingHole_2-5mm, Mounting_Holes:MountingHole_2-5mm, F.Cu at (159.3, 89.4)
- added REF**: MountingHole_2-5mm, Mounting_Holes:MountingHole_2-5mm, F.Cu at (159.6, 125.8)
Other:
- board size 59.4 x 37.3 mm -> 66.7 x 42.2 mm
Changed lines of the file:
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@@
 (kicad_pcb (version 4) (host pcbnew "(2015-11-24 BZR 6329, Git e511afd)-product")
   (general
-    (links 39)
+    (links 0)
     (no_connects 0)
     (area 158.724999 89.874999 218.275001 127.375001)
@@
     (tracks 232)
     (zones 0)
-    (modules 10)
+    (modules 14)
     (nets 26)
   )
@@
   )
   (setup
-    (last_trace_width 0.5)
+    (last_trace_width 0.25)
     (user_trace_width 0.4)
     (user_trace_width 0.5)
@@
     )
   )
-  (gr_line (start 158.8 127.3) (end 158.8 90.05) (layer Edge.Cuts) (width 0.15))
-  (gr_line (start 218.2 127.3) (end 158.8 127.3) (layer Edge.Cuts) (width 0.15))
-  (gr_line (start 218.2 89.95) (end 218.2 127.3) (layer Edge.Cuts) (width 0.15))
-  (gr_line (start 158.8 90.05) (end 218.2 89.95) (layer Edge.Cuts) (width 0.15))
+  (module Mounting_Holes:MountingHole_2-5mm (layer F.Cu)
+    (at 219.4 89.5)
+    (descr "Mounting hole, Befestigungsbohrung, 2,5mm, No Annular, Kein Restring,")
+    (tags "Mounting hole, Befestigungsbohrung, 2,5mm, No Annular, Kein Restring,")
+    (fp_text reference REF** (at 0 -3.50012) (layer F.SilkS)
+      (effects (font (size 1 1) (thickness 0.15)))
+    )
+    (fp_text value MountingHole_2-5mm (at 0.09906 3.59918) (layer F.Fab)
+      (effects (font (size 1 1) (thickness 0.15)))
+    )
+    (fp_circle (center 0 0) (end 2.5 0) (layer Cmts.User) (width 0.381))
+    (pad 1 thru_hole circle (at 0 0) (size 2.5 2.5) (drill 2.5) (layers))
+  )
+  (module Mounting_Holes:MountingHole_2-5mm (layer F.Cu)
+    (at 219.3 125)
+    (descr "Mounting hole, Befestigungsbohrung, 2,5mm, No Annular, Kein Restring,")
+    (tags "Mounting hole, Befestigungsbohrung, 2,5mm, No Annular, Kein Restring,")
+    (fp_text reference REF** (at 0 -3.50012) (layer F.SilkS)
+      (effects (font (size 1 1) (thickness 0.15)))
+    )
+    (fp_text value MountingHole_2-5mm (at 0.09906 3.59918) (layer F.Fab)
+      (effects (font (size 1 1) (thickness 0.15)))
+    )
+    (fp_circle (center 0 0) (end 2.5 0) (layer Cmts.User) (width 0.381))
+    (pad 1 thru_hole circle (at 0 0) (size 2.5 2.5) (drill 2.5) (layers))
+  )
+  (module Mounting_Holes:MountingHole_2-5mm (layer F.Cu)
+    (at 159.3 89.4)
+    (descr "Mounting hole, Befestigungsbohrung, 2,5mm, No Annular, Kein Restring,")
+    (tags "Mounting hole, Befestigungsbohrung, 2,5mm, No Annular, Kein Restring,")
+    (fp_text reference REF** (at 0 -3.50012) (layer F.SilkS)
+      (effects (font (size 1 1) (thickness 0.15)))
+    )
+    (fp_text value MountingHole_2-5mm (at 0.09906 3.59918) (layer F.Fab)
+      (effects (font (size 1 1) (thickness 0.15)))
+    )
+    (fp_circle (center 0 0) (end 2.5 0) (layer Cmts.User) (width 0.381))
+    (pad 1 thru_hole circle (at 0 0) (size 2.5 2.5) (drill 2.5) (layers))
+  )
+  (module Mounting_Holes:MountingHole_2-5mm (layer F.Cu)
+    (at 159.6 125.8)
+    (descr "Mounting hole, Befestigungsbohrung, 2,5mm, No Annular, Kein Restring,")
+    (tags "Mounting hole, Befestigungsbohrung, 2,5mm, No Annular, Kein Restring,")
+    (fp_text reference REF** (at 0 -3.50012) (layer F.SilkS)
+      (effects (font (size 1 1) (thickness 0.15)))
+    )
+    (fp_text value MountingHole_2-5mm (at 0.09906 3.59918) (layer F.Fab)
+      (effects (font (size 1 1) (thickness 0.15)))
+    )
+    (fp_circle (center 0 0) (end 2.5 0) (layer Cmts.User) (width 0.381))
+    (pad 1 thru_hole circle (at 0 0) (size 2.5 2.5) (drill 2.5) (layers))
+  )
+  (gr_line (start 156.4 128.7) (end 156.2 86.5) (layer Edge.Cuts) (width 0.15))
+  (gr_line (start 222.6 128.3) (end 156.4 128.7) (layer Edge.Cuts) (width 0.15))
+  (gr_line (start 222.9 86.5) (end 222.6 128.3) (layer Edge.Cuts) (width 0.15))
+  (gr_line (start 156.2 86.5) (end 222.9 86.5) (layer Edge.Cuts) (width 0.15))
   (segment (start 168.341314 110.85) (end 171.95 110.85) (width 0.5) (layer F.Cu) (net 1))
   (segment (start 171.95 110.85) (end 175.95 106.85) (width 0.5) (layer F.Cu) (net 1))
@@
     (polygon
       (pts
-        (xy 158.8 90.1) (xy 218.1 89.95) (xy 218.2 127.3) (xy 158.8 127.25)
+        (xy 156.1 86.5) (xy 222.9 86.5) (xy 222.5 128.3) (xy 156.4 128.7)
       )
     )
@@
     (polygon
       (pts
-        (xy 158.8 90.05) (xy 218.15 89.95) (xy 218.2 127.25) (xy 158.8 127.25)
+        (xy 156.1 86.5) (xy 222.9 86.5) (xy 222.5 128.3) (xy 156.4 128.7)
       )
     )
