File: led-lamp/led-eight/eight.kicad_pcb (KiCad board)
At the start: 2 copper layers, 61.8 x 61.8 mm, 25 parts, among them U1 RGBLED5050_RGBLED5050, U2 RGBLED5050_RGBLED5050, U3 RGBLED5050_RGBLED5050, U4 RGBLED5050_RGBLED5050, U5 RGBLED5050_RGBLED5050, U6 RGBLED5050_RGBLED5050, U7 RGBLED5050_RGBLED5050, U8 RGBLED5050_RGBLED5050

Commit message: LED lamp use SMD 1206 Resistor
Parts:
- R1, R2, R3, R4, R5, R6, R7, R8: footprint Resistors_ThroughHole:Resistor_Horizontal_RM10mm -> Resistors_SMD:R_1206; moved to F.Cu
- moved R1 4.87 mm to (180.5, 104.7)
- moved R6 4.46 mm to (219.2, 118.8)
- moved R2 4.42 mm to (200.1, 104.3)
- moved R4 4.25 mm to (180.5, 119.3)
- moved R3 4.25 mm to (219.2, 104.1)
- moved R8 4.19 mm to (220.1, 134.8)
- moved R7 3.99 mm to (200.7, 134.8)
- moved R5 3.71 mm to (181.7, 134.5)
Routing:
- net GND: track 155.1 -> 166.1 mm
- net Net-(R5-Pad2): track 6.74 -> 5.98 mm
- net Net-(R8-Pad2): track 6.71 -> 6.04 mm
- net Net-(R4-Pad2): track 6.85 -> 6.20 mm
- net Net-(R2-Pad2): track 6.89 -> 6.24 mm
- net Net-(R6-Pad2): track 6.91 -> 6.29 mm
