File: led-lamp/led-four/four.kicad_pcb (KiCad board)
At the start: 2 copper layers, 59.7 x 59.7 mm, 17 parts, among them U1 RGBLED5050_RGBLED5050, U2 RGBLED5050_RGBLED5050, U3 RGBLED5050_RGBLED5050, U4 RGBLED5050_RGBLED5050

Commit message: LED lamp use SMD 1206 Resistor
Parts:
- R1, R2, R3, R4: footprint Resistors_ThroughHole:Resistor_Horizontal_RM10mm -> Resistors_SMD:R_1206; moved to F.Cu
- moved R2 4.63 mm to (202.3, 110.4)
- moved R1 4.50 mm to (216.8, 124.9)
- moved R4 4.37 mm to (186.2, 125.1)
- moved R3 4.11 mm to (202.9, 138.3)
Routing:
- net GND: track 120.9 -> 145.2 mm
- net +BATT: track 88.1 -> 65.4 mm
- net Net-(R3-Pad2): track 6.77 -> 6.23 mm
