File: led-lamp/led-six/six.kicad_pcb (KiCad board)
At the start: 2 copper layers, 90.1 x 90.1 mm, 17 parts, among them U1 RGBLED5050_RGBLED5050, U2 RGBLED5050_RGBLED5050, U3 RGBLED5050_RGBLED5050, U4 RGBLED5050_RGBLED5050, U5 RGBLED5050_RGBLED5050, U6 RGBLED5050_RGBLED5050

Commit message: LED lamp use SMD 1206 Resistor
Parts:
- R1, R2, R3, R4, R5, R6: footprint Resistors_ThroughHole:Resistor_Horizontal_RM10mm -> Resistors_SMD:R_1206; moved to F.Cu
- moved R4 4.48 mm to (149.0, 116.0)
- moved R6 4.45 mm to (166.6, 140.7)
- moved R2 4.40 mm to (200.8, 85.4)
- moved R1 4.17 mm to (168.3, 85.0)
- moved R3 4.10 mm to (219.3, 116.6)
- moved R5 3.56 mm to (203.9, 141.3)
Routing:
- net +BATT: track 242.7 -> 204.2 mm
- net GND: track 261.8 -> 274.8 mm
- net Net-(R3-Pad2): track 6.57 -> 5.98 mm
