File: test-bench/main/main.kicad_pcb (KiCad board)
At the start: 2 copper layers, 133.7 x 97 mm, 47 parts, among them IC1 ATMEGA128-A, U1 4511N_DIL16, U2 LM2596S_TO263-5, U3 PCF8563, Y1 32khz

Commit message: revisi
Routing:
- net Net-(C-REG1-Pad1): track 12.0 -> 12.6 mm
Changed lines of the file:
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@@
   (general
     (links 175)
-    (no_connects 1)
-    (area 82.714536 32.168809 226.983584 133.57418)
+    (no_connects 0)
+    (area 88.024999 34.924999 221.875001 132.075001)
     (thickness 1.6)
     (drawings 4)
-    (tracks 1756)
+    (tracks 1757)
     (zones 0)
     (modules 47)
@@
   (segment (start 111.7396 96.71858) (end 110.326108 96.71858) (width 0.7) (layer F.Cu) (net 49))
   (segment (start 110.326108 96.71858) (end 107.897868 94.29034) (width 0.7) (layer F.Cu) (net 49))
+  (segment (start 114.18386 52.184989) (end 113.765591 52.603258) (width 0.25) (layer F.Cu) (net 50))
   (segment (start 115.7 51.65) (end 114.718849 51.65) (width 1.1) (layer F.Cu) (net 50))
   (segment (start 114.718849 51.65) (end 114.18386 52.184989) (width 1.1) (layer F.Cu) (net 50))

Commit message: 7 Segment On
Connections:
- IC1 pad 2: /MISO -> /MOSI
- IC1 pad 3: /MOSI -> /MISO
- P-ASP1 pad 5: /MOSI -> /MISO
- P-ASP1 pad 6: /MISO -> /MOSI
Routing:
- net /MOSI: track 11.5 -> 12.3 mm
- net /MISO: track 12.3 -> 11.5 mm
Changed lines of the file:
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@@
       (net 1 "Net-(IC1-Pad1)"))
     (pad 2 smd rect (at -7.7 -5.2 270) (size 1.5 0.55) (layers F.Cu F.Paste F.Mask)
+      (net 3 /MOSI))
+    (pad 3 smd rect (at -7.7 -4.4 270) (size 1.5 0.55) (layers F.Cu F.Paste F.Mask)
       (net 2 /MISO))
-    (pad 3 smd rect (at -7.7 -4.4 270) (size 1.5 0.55) (layers F.Cu F.Paste F.Mask)
-      (net 3 /MOSI))
     (pad 4 smd rect (at -7.7 -3.6 270) (size 1.5 0.55) (layers F.Cu F.Paste F.Mask)
       (net 4 "Net-(IC1-Pad4)"))
@@
       (net 7 /SCK))
     (pad 5 thru_hole oval (at 0 -10.16 270) (size 2.032 1.7272) (drill 1.016) (layers *.Cu *.Mask B.SilkS)
+      (net 2 /MISO))
+    (pad 6 thru_hole oval (at 0 -12.7 270) (size 2.032 1.7272) (drill 1.016) (layers *.Cu *.Mask B.SilkS)
       (net 3 /MOSI))
-    (pad 6 thru_hole oval (at 0 -12.7 270) (size 2.032 1.7272) (drill 1.016) (layers *.Cu *.Mask B.SilkS)
-      (net 2 /MISO))
     (model Pin_Headers.3dshapes/Pin_Header_Straight_1x06.wrl
       (at (xyz 0 -0.25 0))
@@
   (gr_line (start 221.6 35.1) (end 221.8 132) (layer Edge.Cuts) (width 0.15))
   (gr_line (start 88.1 35) (end 221.6 35.1) (layer Edge.Cuts) (width 0.15))
-  (segment (start 160.3875 64.75366) (end 160.3875 63.548998) (width 0.5) (layer F.Cu) (net 2))
-  (segment (start 160.3875 63.548998) (end 160.241931 63.403429) (width 0.5) (layer F.Cu) (net 2))
-  (segment (start 155.918191 69.222969) (end 160.3875 64.75366) (width 0.5) (layer F.Cu) (net 2))
-  (segment (start 155.918191 73.784369) (end 155.918191 69.222969) (width 0.5) (layer F.Cu) (net 2))
-  (segment (start 155.118191 68.773289) (end 157.701931 66.189549) (width 0.5) (layer F.Cu) (net 3))
-  (segment (start 157.701931 66.189549) (end 157.701931 63.403429) (width 0.5) (layer F.Cu) (net 3))
-  (segment (start 155.118191 73.784369) (end 155.118191 68.773289) (width 0.5) (layer F.Cu) (net 3))
+  (segment (start 155.118191 68.773289) (end 157.701931 66.189549) (width 0.5) (layer F.Cu) (net 2))
+  (segment (start 157.701931 66.189549) (end 157.701931 63.403429) (width 0.5) (layer F.Cu) (net 2))
+  (segment (start 155.118191 73.784369) (end 155.118191 68.773289) (width 0.5) (layer F.Cu) (net 2))
+  (segment (start 160.3875 64.75366) (end 160.3875 63.548998) (width 0.5) (layer F.Cu) (net 3))
+  (segment (start 160.3875 63.548998) (end 160.241931 63.403429) (width 0.5) (layer F.Cu) (net 3))
+  (segment (start 155.918191 69.222969) (end 160.3875 64.75366) (width 0.5) (layer F.Cu) (net 3))
+  (segment (start 155.918191 73.784369) (end 155.918191 69.222969) (width 0.5) (layer F.Cu) (net 3))
   (segment (start 148.718191 73.784369) (end 148.718191 69.847169) (width 0.5) (layer F.Cu) (net 7))
   (segment (start 148.718191 69.847169) (end 153.645931 64.919429) (width 0.5) (layer F.Cu) (net 7))
