File: test-bench/main/main.sch (KiCad schematic (older format))
At the start: 35 parts, among them IC1 ATMEGA128-A, U1 4511N_DIL16, U2 LM2596S_TO263-5, U3 PCF8563, Y1 32khz

Commit message: Display Main Controller
Parts:
- added P-LAMP1, P-LAMP2, P-LAMP3, P-LAMP4, P-LAMP5, P-LAMP6, P-LAMP7, P-LAMP8: CONN_02X08, Pin_Headers:Pin_Header_Straight_2x08, symbol CONN_02X08
Connections:
- net GND: now also P-LAMP1.16 (P16), P-LAMP2.16 (P16), P-LAMP3.16 (P16), P-LAMP4.16 (P16), P-LAMP5.16 (P16), P-LAMP6.16 (P16), P-LAMP7.16 (P16), P-LAMP8.16 (P16)
- net LA: now also P-LAMP1.10 (P10), P-LAMP2.10 (P10), P-LAMP3.10 (P10), P-LAMP4.10 (P10), P-LAMP5.10 (P10), P-LAMP6.10 (P10), P-LAMP7.10 (P10), P-LAMP8.10 (P10)
- net LB: now also P-LAMP1.8 (P8), P-LAMP2.8 (P8), P-LAMP3.8 (P8), P-LAMP4.8 (P8), P-LAMP5.8 (P8), P-LAMP6.8 (P8), P-LAMP7.8 (P8), P-LAMP8.8 (P8)
- net LC: now also P-LAMP1.6 (P6), P-LAMP2.6 (P6), P-LAMP3.6 (P6), P-LAMP4.6 (P6), P-LAMP5.6 (P6), P-LAMP6.6 (P6), P-LAMP7.6 (P6), P-LAMP8.6 (P6)
- net LD: now also P-LAMP1.4 (P4), P-LAMP2.4 (P4), P-LAMP3.4 (P4), P-LAMP4.4 (P4), P-LAMP5.4 (P4), P-LAMP6.4 (P4), P-LAMP7.4 (P4), P-LAMP8.4 (P4)
- net LE: now also P-LAMP1.2 (P2), P-LAMP2.2 (P2), P-LAMP3.2 (P2), P-LAMP4.2 (P2), P-LAMP5.2 (P2), P-LAMP6.2 (P2), P-LAMP7.2 (P2), P-LAMP8.2 (P2)
- net LF: now also P-LAMP1.14 (P14), P-LAMP2.14 (P14), P-LAMP3.14 (P14), P-LAMP4.14 (P14), P-LAMP5.14 (P14), P-LAMP6.14 (P14), P-LAMP7.14 (P14), P-LAMP8.14 (P14)
- net LG: now also P-LAMP1.12 (P12), P-LAMP2.12 (P12), P-LAMP3.12 (P12), P-LAMP4.12 (P12), P-LAMP5.12 (P12), P-LAMP6.12 (P12), P-LAMP7.12 (P12), P-LAMP8.12 (P12)
- net VCC: now also P-LAMP1.1 (P1), P-LAMP2.1 (P1), P-LAMP3.1 (P1), P-LAMP4.1 (P1), P-LAMP5.1 (P1), P-LAMP6.1 (P1), P-LAMP7.1 (P1), P-LAMP8.1 (P1)
- net D8-A: now reaches IC1.29 ((ICP1)PD4)
- net D8-A: now also P-LAMP8.9 (P9)
- net D8-B: now reaches IC1.30 ((XCK1)PD5)
- net D8-B: now also P-LAMP8.11 (P11)
- net D8-C: now reaches IC1.31 ((T1)PD6)
- net D8-C: now also P-LAMP8.13 (P13)
- net D8-D: now reaches IC1.32 ((T2)PD7)
- net D8-D: now also P-LAMP8.15 (P15)
- net D7-D: now reaches IC1.34 (PG1(~RD~))
- net D7-D: now also P-LAMP7.9 (P9)
- net D7-C: now reaches IC1.35 ((A8)PC0)
- net D7-C: now also P-LAMP7.11 (P11)
- net D7-B: now reaches IC1.36 ((A9)PC1)
- net D7-B: now also P-LAMP7.13 (P13)
- net D7-A: now reaches IC1.37 ((A10)PC2)
- net D7-A: now also P-LAMP7.15 (P15)
- net D6-D: now reaches IC1.38 ((A11)PC3)
- net D6-D: now also P-LAMP6.9 (P9)
- net D6-C: now reaches IC1.39 ((A12)PC4)
- net D6-C: now also P-LAMP6.11 (P11)
- net D6-B: now reaches IC1.40 ((A13)PC5)
- net D6-B: now also P-LAMP6.13 (P13)
- net D6-A: now reaches IC1.41 ((A14)PC6)
- net D6-A: now also P-LAMP6.15 (P15)
- net D5-C: now reaches IC1.42 ((A15)PC7)
- net D5-C: now also P-LAMP5.11 (P11)
- net D5-B: now reaches IC1.43 (PG2(ALE))
- net D5-B: now also P-LAMP5.13 (P13)
- net D5-A: now reaches IC1.44 ((AD7)PA7)
- net D5-A: now also P-LAMP5.15 (P15)
- net D4-C: now reaches IC1.45 ((AD6)PA6)
- net D4-C: now also P-LAMP4.11 (P11)
- net D4-B: now reaches IC1.46 ((AD5)PA5)
- net D4-B: now also P-LAMP4.13 (P13)
- net D4-A: now reaches IC1.47 ((AD4)PA4)
- net D4-A: now also P-LAMP4.15 (P15)
- net D2-C: now reaches IC1.56 (PF5(ADC5/TMS))
- net D2-C: now also P-LAMP2.11 (P11)
- net D2-B: now reaches IC1.57 (PF4(ADC4/TCK))
- net D2-B: now also P-LAMP2.13 (P13)
- net D2-A: now reaches IC1.58 (PF3(ADC3))
- net D2-A: now also P-LAMP2.15 (P15)
- net D1-C: now reaches IC1.59 (PF2(ADC2))
- net D1-C: now also P-LAMP1.11 (P11)
- net D1-B: now reaches IC1.60 (PF1(ADC1))
- net D1-B: now also P-LAMP1.13 (P13)
- net D1-A: now reaches IC1.61 (PF0(ADC0))
- net D1-A: now also P-LAMP1.15 (P15)
- net D3-A: now reaches IC1.7 (PE5(OC3C/INT5))
- net D3-A: now also P-LAMP3.11 (P11)
- net D3-B: now reaches IC1.8 (PE6(T3/INT6))
- net D3-B: now also P-LAMP3.13 (P13)
- net D3-C: now reaches IC1.9 (PE7(IC3/INT7))
- net D3-C: now also P-LAMP3.15 (P15)

Commit message: 7 Segment On
Connections:
- net MISO: now also IC1.3 (PE1(TXD0/PDO)), P-ASP1.5 (P5); no longer IC1.2 (PE0(RXD0/PDI)), P-ASP1.6 (P6)
- net MOSI: now also IC1.2 (PE0(RXD0/PDI)), P-ASP1.6 (P6); no longer IC1.3 (PE1(TXD0/PDO)), P-ASP1.5 (P5)
Changed lines of the file:
@@
 RST
 Text Label 1750 3650 0    60   ~ 0
+MOSI
+Text Label 1750 3750 0    60   ~ 0
 MISO
-Text Label 1750 3750 0    60   ~ 0
-MOSI
 Text Label 4650 1950 0    60   ~ 0
 SCK
@@
 SCK
 Text Label 1150 1100 0    60   ~ 0
+MISO
+Text Label 1150 1200 0    60   ~ 0
 MOSI
-Text Label 1150 1200 0    60   ~ 0
-MISO
 $Comp
 L LM2596S_TO263-5 U2
