File: rev_rb-pcb/base/rev_rb.sch (KiCad schematic (older format))
At the start: 64 parts, among them CON1 BARREL_JACK, J1 audio-jack, J2 audio-jack, P1 USB_A, Q1 MOSFET-PCHANNELSMD, Q2 MOSFET-NCHANNELSMD, Q3 MOSFET-NCHANNELSMD, U1 STM32F103RB, U2 PC817, U3 PC817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

Commit message: learn sleep mode
Connections:
- net VDD: now also P-BOOT1.1 (P1); no longer U1.13 (VDDA), U7.5 (OUT), U8.2 (OUT)
Changed lines of the file:
@@
 L-LAMP
 Wire Wire Line
-	2550 800  3500 800
+	2550 800  2700 800
+Wire Wire Line
+	2700 800  2900 800
+Wire Wire Line
+	2900 800  3000 800
+Wire Wire Line
+	3000 800  3200 800
 Connection ~ 2900 800
 Connection ~ 3000 800
@@
 	1200 1400 1250 1400
 Wire Wire Line
-	950  1650 950  1850
-Wire Wire Line
-	950  2150 1250 2150
+	950  1650 950  1800
+Wire Wire Line
+	950  1800 950  1850
+Wire Wire Line
+	950  2150 1100 2150
+Wire Wire Line
+	1100 2150 1250 2150
 Wire Wire Line
 	1100 2200 1100 2150
@@
 Connection ~ 950  1800
 Wire Wire Line
-	1250 1700 1250 1850
+	1250 1700 1250 1800
+Wire Wire Line
+	1250 1800 1250 1850
 Wire Wire Line
 	1250 1700 1400 1700
@@
 Connection ~ 1250 1800
 Wire Wire Line
-	2600 4800 3500 4800
+	2600 4800 2700 4800
+Wire Wire Line
+	2700 4800 2900 4800
+Wire Wire Line
+	2900 4800 3000 4800
+Wire Wire Line
+	3000 4800 3200 4800
+Wire Wire Line
+	3200 4800 3500 4800
 Connection ~ 2700 4800
 Connection ~ 2900 4800
@@
 	1300 6350 1300 6750
 Wire Wire Line
-	1250 6750 1800 6750
-Wire Wire Line
-	1250 6250 1700 6250
-Wire Wire Line
-	1300 6250 1300 5900
+	1250 6750 1300 6750
+Wire Wire Line
+	1300 6750 1800 6750
+Wire Wire Line
+	1250 6250 1300 6250
+Wire Wire Line
+	1300 6250 1700 6250
+Wire Wire Line
+	1300 6250 1300 6100
+Wire Wire Line
+	1300 6100 1300 5900
 Wire Wire Line
 	1300 5900 1250 5900
 Wire Wire Line
-	1250 5800 1750 5800
+	1250 5800 1300 5800
+Wire Wire Line
+	1300 5800 1750 5800
 Wire Wire Line
 	1300 5800 1300 5450
@@
 	1300 5350 1300 5250
 Wire Wire Line
-	2100 5150 2700 5150
+	2100 5150 2150 5150
+Wire Wire Line
+	2150 5150 2350 5150
+Wire Wire Line
+	2350 5150 2700 5150
 Connection ~ 2150 5150
 Wire Wire Line
-	2050 5450 2350 5450
+	2050 5450 2150 5450
+Wire Wire Line
+	2150 5450 2350 5450
 Connection ~ 2150 5450
 Wire Wire Line
-	2100 5700 2700 5700
+	2100 5700 2150 5700
+Wire Wire Line
+	2150 5700 2350 5700
+Wire Wire Line
+	2350 5700 2700 5700
 Connection ~ 2150 5700
 Wire Wire Line
-	2050 6000 2350 6000
+	2050 6000 2150 6000
+Wire Wire Line
+	2150 6000 2350 6000
 Connection ~ 2150 6000
 Wire Wire Line
-	1250 5350 1800 5350
-Wire Wire Line
-	2100 6200 2700 6200
+	1250 5350 1300 5350
+Wire Wire Line
+	1300 5350 1800 5350
+Wire Wire Line
+	2100 6200 2150 6200
+Wire Wire Line
+	2150 6200 2350 6200
+Wire Wire Line
+	2350 6200 2700 6200
 Connection ~ 2150 6200
 Wire Wire Line
-	2050 6500 2350 6500
+	2050 6500 2150 6500
+Wire Wire Line
+	2150 6500 2350 6500
 Connection ~ 2150 6500
 Wire Wire Line
-	2100 6750 2700 6750
+	2100 6750 2150 6750
+Wire Wire Line
+	2150 6750 2350 6750
+Wire Wire Line
+	2350 6750 2700 6750
 Connection ~ 2150 6750
 Wire Wire Line
-	2050 7050 2350 7050
+	2050 7050 2150 7050
+Wire Wire Line
+	2150 7050 2350 7050
 Connection ~ 2150 7050
 Wire Wire Line
@@
 	4700 3100 5750 3100
 Wire Wire Line
-	900  2600 900  2850
-Wire Wire Line
-	900  3150 1200 3150
+	900  2600 900  2800
+Wire Wire Line
+	900  2800 900  2850
+Wire Wire Line
+	900  3150 1050 3150
+Wire Wire Line
+	1050 3150 1200 3150
 Wire Wire Line
 	1050 3200 1050 3150
 Connection ~ 1050 3150
 Wire Wire Line
-	1200 2700 1200 2850
+	1200 2700 1200 2800
+Wire Wire Line
+	1200 2800 1200 2850
 Wire Wire Line
 	1700 2700 1200 2700
@@
 	8950 1200 9150 1200
 Wire Wire Line
-	7400 1400 7400 1550
+	7400 1400 7400 1450
+Wire Wire Line
+	7400 1450 7400 1550
 Wire Wire Line
 	7300 1450 7400 1450
 Connection ~ 7400 1450
 Wire Wire Line
-	6600 1450 7000 1450
+	6600 1450 6750 1450
+Wire Wire Line
+	6750 1450 6900 1450
+Wire Wire Line
+	6900 1450 7000 1450
 Connection ~ 6900 1450
 Wire Wire Line
-	6750 1750 7000 1750
+	6750 1750 6900 1750
+Wire Wire Line
+	6900 1750 7000 1750
 Connection ~ 6900 1750
 Connection ~ 6750 1450
@@
 	7050 3000 7250 3000
 Wire Wire Line
-	7050 3750 7300 3750
+	7050 3750 7250 3750
+Wire Wire Line
+	7250 3750 7300 3750
 Wire Wire Line
 	7250 3750 7250 3500
 Connection ~ 7250 3750
 Wire Wire Line
-	7050 4250 9350 4250
+	7050 4250 7300 4250
+Wire Wire Line
+	7300 4250 7700 4250
+Wire Wire Line
+	7700 4250 7800 4250
+Wire Wire Line
+	7800 4250 8250 4250
+Wire Wire Line
+	8250 4250 8950 4250
+Wire Wire Line
+	8950 4250 9200 4250
+Wire Wire Line
+	9200 4250 9350 4250
 Wire Wire Line
 	7050 4250 7050 4050
@@
 Connection ~ 7700 4250
 Wire Wire Line
-	8100 3750 8350 3750
+	8100 3750 8250 3750
+Wire Wire Line
+	8250 3750 8350 3750
 Connection ~ 8250 3750
 Wire Wire Line
-	8950 3500 8950 3800
+	8950 3500 8950 3750
+Wire Wire Line
+	8950 3750 8950 3800
 Wire Wire Line
 	8950 4250 8950 4100
@@
 Connection ~ 9200 4250
 Wire Wire Line
-	9650 4250 9900 4250
+	9650 4250 9800 4250
+Wire Wire Line
+	9800 4250 9900 4250
 Wire Wire Line
 	4700 1700 4900 1700
@@
 	10200 3950 9800 3950
 Wire Wire Line
-	9800 3750 9800 4250
+	9800 3750 9800 3950
+Wire Wire Line
+	9800 3950 9800 4250
 Connection ~ 9800 4250
 Connection ~ 9800 3950
@@
 	9150 1700 9150 1900
 Wire Wire Line
-	9150 1900 9800 1900
+	9150 1900 9500 1900
+Wire Wire Line
+	9500 1900 9800 1900
 Wire Wire Line
 	9800 2300 9500 2300
@@
 Connection ~ 9500 1900
 Wire Wire Line
-	9550 2400 9800 2400
-Wire Wire Line
-	9650 2000 9650 2500
+	9550 2400 9650 2400
+Wire Wire Line
+	9650 2400 9800 2400
+Wire Wire Line
+	9650 2000 9650 2400
+Wire Wire Line
+	9650 2400 9650 2500
 Wire Wire Line
 	9650 2000 9800 2000
@@
 	4700 1800 4900 1800
 Wire Wire Line
-	4100 5700 4350 5700
+	4100 5700 4200 5700
+Wire Wire Line
+	4200 5700 4350 5700
 Wire Wire Line
 	4200 5300 4200 5400
@@
 	4700 4400 4850 4400
 Wire Wire Line
-	4100 6450 4350 6450
+	4100 6450 4200 6450
+Wire Wire Line
+	4200 6450 4350 6450
 Wire Wire Line
 	4200 6050 4200 6150
@@
 	3750 6900 3700 6900
 Wire Wire Line
-	3600 7100 3750 7100
+	3600 7100 3700 7100
+Wire Wire Line
+	3700 7100 3750 7100
 Wire Wire Line
 	3700 7100 3700 7150
@@
 	3600 7300 3600 7100
 Connection ~ 3700 7100
-Connection ~ 4000 6700
 Wire Wire Line
 	5200 5250 5000 5250
@@
 	5600 5250 5650 5250
 Wire Wire Line
-	5650 5250 5650 5950
+	5650 5250 5650 5450
+Wire Wire Line
+	5650 5450 5650 5650
+Wire Wire Line
+	5650 5650 5650 5850
+Wire Wire Line
+	5650 5850 5650 5950
 Wire Wire Line
 	5600 5850 5650 5850
@@
 	4700 3500 4900 3500
 Wire Wire Line
-	5600 6250 5600 6700
+	5600 6250 5600 6450
+Wire Wire Line
+	5600 6450 5600 6650
+Wire Wire Line
+	5600 6650 5600 6700
 Connection ~ 5600 6450
 Connection ~ 5600 6650
@@
 	1    0    0    -1
 $EndComp
-Connection ~ 3200 800
 $Comp
 L GNDPWR #PWR7
@@
 U 1 1 56CBBF0A
 P 6350 5000
-F 0 "U7" H 6350 5000 0   0001 C CNN
-F 1 "MIC5219BM5_SOT23-5" H 6350 5000 0   0001 C CNN
+F 0 "U7" H 6350 5000 60  0001 C CNN
+F 1 "MIC5219BM5_SOT23-5" H 6350 5000 60  0001 C CNN
 F 2 "" H 6350 5000 60  0000 C CNN
 F 3 "" H 6350 5000 60  0000 C CNN
@@
 	6450 5500 6450 5400
 $Comp
-L VDD #PWR33
-U 1 1 56CC324A
-P 6850 4800
-F 0 "#PWR33" H 6850 4650 50  0001 C CNN
-F 1 "VDD" H 6850 4950 50  0000 C CNN
-F 2 "" H 6850 4800 50  0000 C CNN
-F 3 "" H 6850 4800 50  0000 C CNN
-	1    6850 4800
-	1    0    0    -1
-$EndComp
-Wire Wire Line
-	6750 4800 6850 4800
-$Comp
 L XC63FPM_SOT23 U8
 U 1 1 56CC57BA
 P 6450 5800
-F 0 "U8" H 6450 5800 0   0001 C CNN
-F 1 "XC63FPM_SOT23" H 6450 5800 0   0001 C CNN
+F 0 "U8" H 6450 5800 60  0001 C CNN
+F 1 "XC63FPM_SOT23" H 6450 5800 60  0001 C CNN
 F 2 "" H 6450 5800 60  0000 C CNN
 F 3 "" H 6450 5800 60  0000 C CNN
 	1    6450 5800
-	1    0    0    -1
-$EndComp
-$Comp
-L VDD #PWR34
-U 1 1 56CC58FA
-P 6850 5800
-F 0 "#PWR34" H 6850 5650 50  0001 C CNN
-F 1 "VDD" H 6850 5950 50  0000 C CNN
-F 2 "" H 6850 5800 50  0000 C CNN
-F 3 "" H 6850 5800 50  0000 C CNN
-	1    6850 5800
 	1    0    0    -1
 $EndComp
@@
 $EndComp
 Wire Wire Line
-	6850 5800 6750 5800
-Wire Wire Line
 	6450 6100 6450 6200
 Wire Wire Line
 	6150 5800 6050 5800
+Wire Wire Line
+	1200 1200 1250 1200
 $EndSCHEMATC
