File: rev_rb-pcb/test1/rev_rb.kicad_pcb (KiCad board)
At the start: 2 copper layers, 50 parts, among them CON1 BARREL_JACK, J1 audio-jack, J2 audio-jack, P1 CONN_01X03, P2 CONN_01X03, Q1 MOSFET-PCHANNELSMD, Q2 MOSFET-NCHANNELSMD, U1 STM32F103RB, U2 CNY17-4, U3 CNY17-4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

Commit message: begins
Parts:
- removed C1: C, Capacitors_SMD:C_0805
- removed D-ADC-PV1: D, Diodes_SMD:SMA_Standard
- added R5: 330, Resistors_SMD:R_0805, F.Cu at (216.5, 116.3)
- added TP1: TEST-POINT2, tespad:SparkFun-PAD.03X.05, F.Cu at (46.5, 150.1)
- added TP10: TEST-POINT2, tespad:SparkFun-PAD.03X.05, F.Cu at (165.4, 91.2)
- added TP11: TEST-POINT2, tespad:SparkFun-PAD.03X.05, F.Cu at (176.9, 110.4)
- added TP12: TEST-POINT2, tespad:SparkFun-PAD.03X.05, F.Cu at (183.3, 106.7)
- added TP2: TEST-POINT2, tespad:SparkFun-PAD.03X.05, F.Cu at (106.1, 142.8)
- added TP3: TEST-POINT2, tespad:SparkFun-PAD.03X.05, F.Cu at (168.0, 98.8)
- added TP4: TEST-POINT2, tespad:SparkFun-PAD.03X.05, F.Cu at (176.7, 98.0)
- added TP5: TEST-POINT2, tespad:SparkFun-PAD.03X.05, F.Cu at (176.5, 104.1)
- added TP6: TEST-POINT2, tespad:SparkFun-PAD.03X.05, F.Cu at (173.6, 107.9)
- added TP7: TEST-POINT2, tespad:SparkFun-PAD.03X.05, F.Cu at (147.7, 142.5)
- added TP8: TEST-POINT2, tespad:SparkFun-PAD.03X.05, F.Cu at (125.7, 142.6)
- added TP9: TEST-POINT2, tespad:SparkFun-PAD.03X.05, F.Cu at (167.4, 94.7)
- added U4: PC817, Housings_DIP:DIP-4_W7.62mm, F.Cu at (63.6, 150.1)
- added U5: 10-XX_B3F-10XX, switch-omron:B3F-10XX, F.Cu at (64.5, 94.8)
- R1: value 10k -> 330
- R2: value 33k -> 10k
- U2, U3: value CNY17-4 -> PC817; footprint cny17:SMD-6 -> Housings_DIP:DIP-4_W7.62mm
- moved Q1 133.1 mm to (58.7, 141.9), turned to 90 degrees
- moved J1 123.9 mm to (224.1, 141.3), turned to 90 degrees
- moved J2 114.6 mm to (215.4, 141.3), turned to 90 degrees
- moved R1 108.5 mm to (53.6, 157.7), turned to 90 degrees
- moved D1 106.9 mm to (221.6, 128.4), turned to 180 degrees
- moved U2 105.8 mm to (54.8, 154.2), turned to 90 degrees
- moved R2 91.4 mm to (66.8, 146.0)
- moved U6 85.9 mm to (64.6, 86.8)
- moved C4 82.6 mm to (65.9, 105.6)
- moved R3 80.7 mm to (69.9, 86.8), turned to 90 degrees
- moved R4 79.4 mm to (69.8, 94.8), turned to 270 degrees
- moved D6 74.2 mm to (215.4, 137.0), turned to 270 degrees
- moved U3 69.1 mm to (215.7, 120.8)
- moved C-XTAL1 68.1 mm to (86.7, 76.4), turned to 270 degrees
- moved C-XTAL2 66.2 mm to (86.6, 81.6), turned to 90 degrees
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Connections:
- C4 pad 1: Net-(C4-Pad1) -> /ADC-DIM
- CON1 pad 1: Net-(CON1-Pad1) -> /V-PV
- Q1 pad 2: Net-(D-ADC-PV1-Pad1) -> /V-PV
- R1 pad 1: /ADC-PV -> /CON-PV
- R1 pad 2: GND -> Net-(R1-Pad2)
- R2 pad 1: Net-(CON1-Pad1) -> /V-PV
- R2 pad 2: /ADC-PV -> Net-(R2-Pad2)
- U1 pad 14: /ADC-BATT1 -> /IND-PV
- U1 pad 15: /ADC-BATT2 -> /ADC-BATT1
- U1 pad 16: /ADC-PV -> /ADC-BATT2
- U2 pad 1: /CON-PV -> Net-(R1-Pad2)
- U2 pad 3: (no net) -> Net-(Q1-Pad1)
- U2 pad 4: Net-(Q1-Pad1) -> /V-PV
- U3 pad 1: /CON-LAMP -> Net-(R5-Pad2)
- U3 pad 3: (no net) -> Net-(Q2-Pad1)
- U3 pad 4: Net-(Q2-Pad1) -> Net-(D1-Pad1)
Routing:
- net GND: track 0.00 -> 83.9 mm
- net +6V: track 0.00 -> 10.2 mm
- net /ADC-BATT2: track 0.00 -> 6.88 mm
- net /ADC-BATT1: track 0.00 -> 6.36 mm
- net GNDPWR: track 0.00 -> 5.85 mm
- net Net-(BATT1-Pad1): track 0.00 -> 5.67 mm
- net Net-(BATT3-Pad1): track 0.00 -> 5.65 mm
- net +BATT: track 0.00 -> 4.70 mm

Commit message: progress
Parts:
- CON1: footprint Connect:BARREL_JACK -> Connect:JACK_ALIM; moved to B.Cu
- J1, J2, P-BOOT1, P-COMM1, P-MIC1, P-VDD1, P-XC1, P1, P2, U2, U3, U4, U5, U6, VDD-VDDA1, Y1: moved to B.Cu
- Q1, Q2: footprint TO_SOT_Packages_SMD:TO-263-3Lead -> Power_Integrations:TO-220; moved to B.Cu
- moved Q2 121.3 mm to (107.7, 131.1)
- moved D1 118.0 mm to (104.2, 140.1), turned to 270 degrees
- moved R5 109.7 mm to (109.7, 141.6)
- moved U3 108.0 mm to (110.2, 143.9), turned to 90 degrees
- moved TP5 104.6 mm to (71.9, 102.0), turned to 180 degrees
- moved TP11 103.1 mm to (75.3, 92.6), turned to 90 degrees
- moved TP6 102.1 mm to (71.9, 99.1), turned to 180 degrees
- moved J1 102.1 mm to (123.7, 123.1), turned to 180 degrees
- moved D6 96.2 mm to (119.6, 145.6), turned to 0 degrees
- moved J2 92.0 mm to (123.7, 132.6), turned to 180 degrees
- moved TP1 89.8 mm to (124.4, 105.4), turned to 180 degrees
- moved TP4 88.2 mm to (90.1, 115.2), turned to 90 degrees
- moved CON1 86.3 mm to (124.5, 112.0), turned to 180 degrees
- moved TP3 82.8 mm to (85.2, 95.2), turned to 90 degrees
- moved R1 81.3 mm to (113.6, 102.8), turned to 180 degrees
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Routing:
- net +BATT: track 4.70 -> 126.4 mm
- net GND: track 83.9 -> 200.9 mm, vias 0 -> 2
- net /CON-LAMP: track 0.00 -> 93.6 mm
- net VDD: track 0.00 -> 86.5 mm
- net /ADC-LAMP: track 0.00 -> 80.4 mm, vias 0 -> 4
- net /V-PV: track 0.00 -> 55.8 mm
- net /ADC-BATT2: track 6.88 -> 45.3 mm
- net /ADC-DIM: track 0.00 -> 37.5 mm, vias 0 -> 2
- net Net-(J1-Pad2): track 0.00 -> 28.2 mm
- net /IND-PV: track 0.00 -> 26.8 mm, vias 0 -> 2
- net /CON-PV: track 0.00 -> 22.6 mm, vias 0 -> 2
- net /NRST: track 0.00 -> 21.9 mm
- net /ADC-BATT1: track 6.36 -> 23.6 mm
- net /BTN-USER: track 0.00 -> 16.5 mm
- net Net-(Q1-Pad1): track 0.00 -> 13.6 mm
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
Commit message: progress
Parts:
- moved D6 59.5 mm to (175.8, 125.9)
- moved RA7 59.5 mm to (146.0, 104.9)
- moved U7 59.5 mm to (128.7, 92.6)
- moved BATT2 59.5 mm to (141.8, 93.0)
- moved BATT3 59.5 mm to (141.8, 103.5)
- moved C-XTAL1 59.5 mm to (147.7, 59.4)
- moved CA1 59.5 mm to (148.4, 83.1)
- moved CA3 59.5 mm to (148.2, 105.0)
- moved D1 59.5 mm to (160.3, 120.3)
- moved D10 59.5 mm to (162.9, 53.4)
- moved D11 59.5 mm to (159.2, 53.5)
- moved D13 59.5 mm to (152.9, 53.5)
- moved D8 59.5 mm to (167.2, 53.4)
- moved J1 59.5 mm to (179.8, 103.3)
- moved P-BOOT1 59.5 mm to (154.3, 49.3)
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Routing:
- net GND: track 200.9 -> 394.2 mm, vias 2 -> 14
- net VDD: track 86.5 -> 269.4 mm, vias 0 -> 4
- net +3V3: track 9.32 -> 104.5 mm, vias 0 -> 6
- net GNDPWR: track 18.5 -> 62.2 mm, vias 0 -> 2
- net +6V: track 21.5 -> 34.2 mm, vias 0 -> 2
- net /ADC-LAMP: track 80.4 -> 82.0 mm
- net +BATT: track 126.4 -> 127.9 mm
Other:
- board outline added: 68 x 86 mm
- net class Default: via_dia 0.6 -> 1.2; via_drill 0.4 -> 0.8
