File: rev_rb-pcb/test1/rev_rb.kicad_pcb (KiCad board)
At the start: 2 copper layers, 65.9 x 84.5 mm, 60 parts, among them CON1 BARREL_JACK, J1 audio-jack, P1 CONN_01X03, P2 CONN_01X03, Q1 MOSFET-PCHANNELSMD, Q2 MOSFET-NCHANNELSMD, U1 STM32F103RB, U2 PC817, U3 PC817, U4 PC817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

Commit message: new print
Routing:
- net VDD: track 200.3 -> 216.8 mm, vias 10 -> 12
Other:
- board text added: "PSHS"
- board text added: "v0.4"
Changed lines of the file:
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@@
   (general
     (links 120)
-    (no_connects 2)
-    (area 88.545199 59.487599 154.583601 144.118801)
+    (no_connects 1)
+    (area 88.545199 59.487599 156.282889 144.118801)
     (thickness 1.6)
-    (drawings 4)
-    (tracks 586)
+    (drawings 6)
+    (tracks 596)
     (zones 0)
     (modules 60)
@@
       (rotate (xyz 0 0 0))
     )
+  )
+  (gr_text v0.4 (at 98.7552 73.6854) (layer F.Cu)
+    (effects (font (size 1.5 1.5) (thickness 0.3)))
+  )
+  (gr_text PSHS (at 98.425 66.0146) (layer F.Cu)
+    (effects (font (size 2 2) (thickness 0.5)))
   )
   (gr_line (start 88.5952 144.0688) (end 88.7222 59.5376) (layer Edge.Cuts) (width 0.1))
@@
   (segment (start 97.88398 106.53522) (end 97.88398 103.89362) (width 0.4) (layer F.Cu) (net 24))
   (segment (start 97.88398 103.89362) (end 97.85858 103.86822) (width 0.4) (layer F.Cu) (net 24))
+  (segment (start 132.69976 77.1906) (end 132.69976 73.7362) (width 0.25) (layer F.Cu) (net 25))
+  (segment (start 131.4704 73.8124) (end 131.770399 73.512401) (width 0.25) (layer F.Cu) (net 25))
+  (segment (start 132.69976 73.7362) (end 132.69976 72.2884) (width 0.25) (layer F.Cu) (net 25))
+  (segment (start 131.770399 73.512401) (end 132.475961 73.512401) (width 0.25) (layer F.Cu) (net 25))
+  (segment (start 132.475961 73.512401) (end 132.69976 73.7362) (width 0.25) (layer F.Cu) (net 25))
+  (via (at 131.4704 73.8124) (size 1.4) (drill 0.8) (layers F.Cu B.Cu) (net 25))
+  (segment (start 119.507 73.8124) (end 131.4704 73.8124) (width 0.25) (layer B.Cu) (net 25))
+  (segment (start 120.43656 73.8124) (end 119.507 73.8124) (width 0.25) (layer F.Cu) (net 25))
+  (via (at 119.507 73.8124) (size 1.4) (drill 0.8) (layers F.Cu B.Cu) (net 25))
+  (segment (start 121.55812 75.53396) (end 121.55812 74.93396) (width 0.25) (layer F.Cu) (net 25))
+  (segment (start 121.55812 74.93396) (end 120.43656 73.8124) (width 0.25) (layer F.Cu) (net 25))
   (segment (start 129.05812 78.14238) (end 129.71654 77.48396) (width 0.25) (layer F.Cu) (net 25))
   (segment (start 129.71654 77.48396) (end 131.00812 77.48396) (width 0.25) (layer F.Cu) (net 25))
@@
   (segment (start 132.69976 72.2884) (end 133.16204 71.82612) (width 0.25) (layer F.Cu) (net 25))
   (segment (start 133.16204 71.82612) (end 134.7216 71.82612) (width 0.25) (layer F.Cu) (net 25))
-  (segment (start 132.69976 77.1906) (end 132.69976 72.2884) (width 0.25) (layer F.Cu) (net 25))
   (segment (start 132.4064 77.48396) (end 132.69976 77.1906) (width 0.25) (layer F.Cu) (net 25))
   (segment (start 131.00812 77.48396) (end 132.4064 77.48396) (width 0.25) (layer F.Cu) (net 25))

Commit message: try again
Parts:
- moved C4 3.05 mm to (128.3, 96.4)
- moved JP2 3.05 mm to (124.6, 99.5)
- moved TP11 3.05 mm to (125.0, 96.4)
- moved P-COMM1 1.66 mm to (136.3, 72.2)
- moved JP1 0.42 mm to (105.4, 130.8)
- moved TP1 0.42 mm to (101.9, 133.5)
- moved TP2 0.42 mm to (101.9, 128.2)
Routing:
- net VDD: track 216.8 -> 270.8 mm, vias 12 -> 16
- net GND: track 313.9 -> 362.8 mm, vias 4 -> 8
- net /CON-LAMP: track 26.1 -> 53.5 mm
- net +6V: track 47.2 -> 57.9 mm, vias 2 -> 0
- net /CON-PV: track 76.1 -> 83.9 mm, vias 0 -> 2
- net +BATT: track 207.6 -> 203.8 mm, vias 6 -> 4
- net GNDPWR: track 55.9 -> 59.5 mm
- net /ADC-BATT2: track 41.7 -> 44.7 mm
- net Net-(P-COMM1-Pad3): track 9.55 -> 12.4 mm
- net +3V3: track 94.1 -> 92.2 mm
- net /ADC-DIM: track 23.7 -> 22.1 mm
- net Net-(P-COMM1-Pad4): track 3.94 -> 5.43 mm
- net Net-(J1-Pad2): track 21.1 -> 19.7 mm
- net /ADC-LAMP: track 45.8 -> 46.7 mm
- net /NRST: track 22.1 -> 22.7 mm
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Other:
- board size 65.9 x 84.5 mm -> 67.2 x 84.9 mm
- board text removed: "PSHS"
- board text removed: "v0.4"

Commit message: progress
Connections:
- net Net-(P-COMM1-Pad3) renamed /TX
- net Net-(P-COMM1-Pad4) renamed /RX

Commit message: standby mode
Connections:
- U1 pad 14: /ADC-BATT1 -> /IND-PV
- U1 pad 21: /IND-PV -> /ADC-BATT1
Routing:
- net /IND-PV: track 96.1 -> 45.8 mm
- net /ADC-BATT1: track 22.9 -> 67.9 mm
Changed lines of the file:
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@@
   (general
     (links 120)
-    (no_connects 0)
-    (area 88.399999 59.249999 156.050001 144.550001)
+    (no_connects 2)
+    (area 88.399999 59.249999 156.282889 144.550001)
     (thickness 1.6)
     (drawings 4)
-    (tracks 706)
+    (tracks 718)
     (zones 0)
     (modules 60)
@@
       (net 24 +3V3))
     (pad 14 smd rect (at -5.7 2.75) (size 1.5 0.3) (layers F.Cu F.Paste F.Mask)
-      (net 10 /ADC-BATT1))
+      (net 39 /IND-PV))
     (pad 15 smd rect (at -5.7 3.25) (size 1.5 0.3) (layers F.Cu F.Paste F.Mask)
       (net 11 /ADC-BATT2))
@@
       (net 47 /ADC-USB))
     (pad 21 smd rect (at -1.75 5.7 90) (size 1.5 0.3) (layers F.Cu F.Paste F.Mask)
-      (net 39 /IND-PV))
+      (net 10 /ADC-BATT1))
     (pad 22 smd rect (at -1.25 5.7 90) (size 1.5 0.3) (layers F.Cu F.Paste F.Mask)
       (net 48 "Net-(U1-Pad22)"))
@@
   (segment (start 127.29664 96.35824) (end 127.29664 99.37356) (width 0.45) (layer F.Cu) (net 9))
   (segment (start 127.29664 99.37356) (end 127.18068 99.48952) (width 0.45) (layer F.Cu) (net 9))
-  (segment (start 117.45 90.05) (end 117.45 97.85) (width 0.45) (layer F.Cu) (net 10))
-  (segment (start 117.45 97.85) (end 116.56568 98.73432) (width 0.45) (layer F.Cu) (net 10))
+  (segment (start 147.1 121.625) (end 147.1 124.15) (width 0.45) (layer F.Cu) (net 10))
+  (segment (start 147.1 121.625) (end 147.175 121.7) (width 0.45) (layer F.Cu) (net 10))
+  (segment (start 150.075 118.65) (end 147.1 121.625) (width 0.45) (layer F.Cu) (net 10))
+  (segment (start 150.075 104.2) (end 150.075 118.65) (width 0.45) (layer F.Cu) (net 10))
+  (segment (start 149.925 104.05) (end 150.075 104.2) (width 0.45) (layer F.Cu) (net 10))
+  (segment (start 149 103.125) (end 149.925 104.05) (width 0.45) (layer F.Cu) (net 10))
+  (segment (start 146.025 100.15) (end 149 103.125) (width 0.45) (layer F.Cu) (net 10))
+  (segment (start 146.025 98.225) (end 146.025 100.15) (width 0.45) (layer F.Cu) (net 10))
+  (segment (start 145.375 97.575) (end 146.025 98.225) (width 0.45) (layer F.Cu) (net 10))
+  (segment (start 141.55 93.75) (end 145.375 97.575) (width 0.45) (layer F.Cu) (net 10))
+  (segment (start 141.45 93.75) (end 141.55 93.75) (width 0.45) (layer F.Cu) (net 10))
+  (segment (start 141.45 93.75) (end 141.65 93.75) (width 0.45) (layer F.Cu) (net 10))
+  (segment (start 117.31752 98.81616) (end 118.35384 99.85248) (width 0.45) (layer F.Cu) (net 10))
+  (segment (start 126.2 93.75) (end 141.45 93.75) (width 0.45) (layer F.Cu) (net 10))
+  (segment (start 123.55812 86.93396) (end 123.55812 93.00812) (width 0.25) (layer F.Cu) (net 10))
+  (segment (start 123.55812 93.00812) (end 124.3 93.75) (width 0.25) (layer F.Cu) (net 10))
+  (segment (start 124.3 93.75) (end 126.2 93.75) (width 0.25) (layer F.Cu) (net 10))
+  (segment (start 126.2 93.75) (end 126.35 93.75) (width 0.25) (layer F.Cu) (net 10))
+  (segment (start 117.475 97.739428) (end 117.475 97.125) (width 0.45) (layer F.Cu) (net 10))
+  (segment (start 116.56568 98.81616) (end 116.56568 98.648748) (width 0.45) (layer F.Cu) (net 10))
+  (segment (start 116.56568 98.648748) (end 117.475 97.739428) (width 0.45) (layer F.Cu) (net 10))
   (segment (start 116.56568 98.73432) (end 116.56568 98.81616) (width 0.45) (layer F.Cu) (net 10))
-  (segment (start 117.15 89.75) (end 117.45 90.05) (width 0.25) (layer F.Cu) (net 10))
-  (segment (start 117.15 89.5) (end 117.15 89.75) (width 0.25) (layer F.Cu) (net 10))
-  (segment (start 117.15 85.16926) (end 117.15 89.5) (width 0.25) (layer F.Cu) (net 10))
-  (segment (start 119.60812 83.98396) (end 118.3353 83.98396) (width 0.25) (layer F.Cu) (net 10))
-  (segment (start 118.3353 83.98396) (end 117.15 85.16926) (width 0.25) (layer F.Cu) (net 10))
   (segment (start 116.56568 98.81616) (end 117.31752 98.81616) (width 0.45) (layer F.Cu) (net 10))
-  (segment (start 117.31752 98.81616) (end 118.35384 99.85248) (width 0.45) (layer F.Cu) (net 10))
   (segment (start 116.56568 98.81616) (end 114.67084 98.81616) (width 0.45) (layer F.Cu) (net 10))
   (segment (start 114.67084 98.81616) (end 114.48288 98.6282) (width 0.45) (layer F.Cu) (net 10))
@@
   (segment (start 128.6002 109.5452) (end 127.1574 109.5452) (width 0.45) (layer F.Cu) (net 38))
   (segment (start 127.1574 109.5452) (end 126.8984 109.8042) (width 0.45) (layer F.Cu) (net 38))
-  (segment (start 126.2 93.75) (end 141.45 93.75) (width 0.45) (layer F.Cu) (net 39))
-  (segment (start 123.55812 86.93396) (end 123.55812 93.00812) (width 0.25) (layer F.Cu) (net 39))
-  (segment (start 123.55812 93.00812) (end 124.3 93.75) (width 0.25) (layer F.Cu) (net 39))
-  (segment (start 124.3 93.75) (end 126.2 93.75) (width 0.25) (layer F.Cu) (net 39))
-  (segment (start 126.2 93.75) (end 126.35 93.75) (width 0.25) (layer F.Cu) (net 39))
-  (segment (start 123.825 136.625) (end 123.825 134.6327) (width 0.45) (layer F.Cu) (net 39))
-  (segment (start 124.2 137) (end 123.825 136.625) (width 0.45) (layer F.Cu) (net 39))
-  (segment (start 140.45 137) (end 124.2 137) (width 0.45) (layer F.Cu) (net 39))
-  (segment (start 147.05 130.4) (end 140.45 137) (width 0.45) (layer F.Cu) (net 39))
-  (segment (start 147.05 121.4) (end 147.05 130.4) (width 0.45) (layer F.Cu) (net 39))
-  (segment (start 149.95 103.9) (end 149.95 118.5) (width 0.45) (layer F.Cu) (net 39))
-  (segment (start 145.95 99.9) (end 149.95 103.9) (width 0.45) (layer F.Cu) (net 39))
-  (segment (start 149.95 118.5) (end 147.05 121.4) (width 0.45) (layer F.Cu) (net 39))
-  (segment (start 145.95 98.25) (end 145.95 99.9) (width 0.45) (layer F.Cu) (net 39))
-  (segment (start 141.45 93.75) (end 145.95 98.25) (width 0.45) (layer F.Cu) (net 39))
+  (segment (start 147.025 130.5) (end 147.025 127.35) (width 0.45) (layer F.Cu) (net 39))
+  (segment (start 143.25 134.275) (end 147.025 130.5) (width 0.45) (layer F.Cu) (net 39))
+  (segment (start 140.4 137.125) (end 143.25 134.275) (width 0.45) (layer F.Cu) (net 39))
+  (segment (start 125.4 137.125) (end 140.4 137.125) (width 0.45) (layer F.Cu) (net 39))
+  (segment (start 124.969275 136.675) (end 124.969275 136.694275) (width 0.45) (layer F.Cu) (net 39))
+  (segment (start 124.969275 136.694275) (end 125.4 137.125) (width 0.45) (layer F.Cu) (net 39))
+  (segment (start 123.825 134.6327) (end 123.825 135.530725) (width 0.45) (layer F.Cu) (net 39))
+  (segment (start 123.825 135.530725) (end 124.969275 136.675) (width 0.45) (layer F.Cu) (net 39))
   (segment (start 123.825 134.6327) (end 121.7676 134.6327) (width 0.45) (layer F.Cu) (net 39))
   (segment (start 121.7676 134.6327) (end 121.6533 134.747) (width 0.45) (layer F.Cu) (net 39))
+  (segment (start 117.45 90.05) (end 117.45 95.05) (width 0.45) (layer F.Cu) (net 39))
+  (segment (start 117.15 89.75) (end 117.45 90.05) (width 0.25) (layer F.Cu) (net 39))
+  (segment (start 117.15 89.5) (end 117.15 89.75) (width 0.25) (layer F.Cu) (net 39))
+  (segment (start 117.15 85.16926) (end 117.15 89.5) (width 0.25) (layer F.Cu) (net 39))
+  (segment (start 119.60812 83.98396) (end 118.3353 83.98396) (width 0.25) (layer F.Cu) (net 39))
+  (segment (start 118.3353 83.98396) (end 117.15 85.16926) (width 0.25) (layer F.Cu) (net 39))
   (segment (start 131.00812 80.48396) (end 134.63396 80.48396) (width 0.25) (layer F.Cu) (net 73))
   (segment (start 134.63396 80.48396) (end 135.35 81.2) (width 0.25) (layer F.Cu) (net 73))
