File: rev_rb-pcb/test1/rev_rb.sch (KiCad schematic (older format))
At the start: 50 parts, among them CON1 BARREL_JACK, J1 audio-jack, J2 audio-jack, P1 CONN_01X03, P2 CONN_01X03, Q1 MOSFET-PCHANNELSMD, Q2 MOSFET-NCHANNELSMD, U1 STM32F103RB, U2 CNY17-4, U3 CNY17-4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

Commit message: begins
Parts:
- removed C1: C, Capacitors_SMD:C_0805, symbol C
- removed D-ADC-PV1: D, Diodes_SMD:SMA_Standard, symbol D
- removed U2, U3: CNY17-4, cny17:SMD-6, symbol CNY17-4
- removed unit 2 of U6
- added R5: 330, Resistors_SMD:R_0805, symbol R
- added TP1, TP10, TP11, TP12, TP2, TP3, TP4, TP5, TP6, TP7, TP8, TP9: TEST-POINT2, tespad:SparkFun-PAD.03X.05, symbol TEST-POINT2
- added U2, U3, U4: PC817, Housings_DIP:DIP-4_W7.62mm, symbol PC817
- added U5: 10-XX_B3F-10XX, switch-omron:B3F-10XX, symbol 10-XX_B3F-10XX
- R1: value 10k -> 330
- R2: value 33k -> 10k
Connections:
- net +3V3: now also TP6.1
- net +6V: now also TP4.1
- net +BATT: now also TP3.1
- net ADC-BATT1: now also U1.15 (USART2_RTS/ADC12_IN1/TIM2_CH2/PA1), TP7.1; no longer U1.14 (WKUP/USART2_CTS/ADC12_IN0/TIM2_CH1_ETR/PA0)
- net ADC-BATT2: now also U1.16 (USART2_TX/ADC12_IN2/TIM2_CH3/PA2), TP8.1; no longer U1.15 (USART2_RTS/ADC12_IN1/TIM2_CH2/PA1)
- net ADC-DIM: now also C4.1, TP11.1
- net ADC-LAMP: now also TP10.1
- net BTN-USER: now also U5.3 (P), U5.4 (P1)
- net CON-LAMP: now also R5.1
- net CON-PV: now also R1.1
- net GND: now also TP2.1, U2.2, U3.2, U4.2, U5.1 (S), U5.2 (S1); no longer R1.2
- net GNDPWR: now also TP1.1
- net VDD: now also TP5.1, U4.4
- net V-PV: now reaches CON1.1, R2.1
- net V-PV: now also Q1.2 (S), TP9.1, U2.4
- net at Q1.1 (G): now also U2.3
- net at Q2.1 (G): now also U3.3
- net at D1.1 (K), Q2.3 (D): now also U3.4
- removed net ADC-PV: R1.1, R2.2, U1.16 (USART2_TX/ADC12_IN2/TIM2_CH3/PA2)
- new net: R1.2, U2.1
- new net: R5.2, U3.1
- new net: R2.2, U4.1
- new net IND-PV: TP12.1, U1.14 (WKUP/USART2_CTS/ADC12_IN0/TIM2_CH1_ETR/PA0), U4.3
Other:
- moved on the sheet: D1, D6, J1, J2, Q2

Commit message: progress
Parts:
- CON1: footprint Connect:BARREL_JACK -> Connect:JACK_ALIM
- Q1, Q2: footprint TO_SOT_Packages_SMD:TO-263-3Lead -> Power_Integrations:TO-220
Changed lines of the file:
@@
 F 0 "CON1" H 8000 1350 50  0000 C CNN
 F 1 "BARREL_JACK" H 8000 900 50  0000 C CNN
-F 2 "Connect:BARREL_JACK" H 8000 1100 50  0001 C CNN
+F 2 "Connect:JACK_ALIM" H 8000 1100 50  0001 C CNN
 F 3 "" H 8000 1100 50  0000 C CNN
 	1    8000 1100
@@
 F 0 "Q1" H 7950 2300 50  0000 L BNN
 F 1 "MOSFET-PCHANNELSMD" H 7950 1950 50  0000 L BNN
-F 2 "TO_SOT_Packages_SMD:TO-263-3Lead" H 8450 2150 50  0001 C CNN
+F 2 "Power_Integrations:TO-220" H 8450 2150 50  0001 C CNN
 F 3 "" H 7900 2150 60  0000 C CNN
 	1    7900 2150
@@
 F 0 "Q2" H 9800 1750 50  0000 L BNN
 F 1 "MOSFET-NCHANNELSMD" H 9800 1400 50  0000 L BNN
-F 2 "TO_SOT_Packages_SMD:TO-263-3Lead" H 10300 1600 50  0001 C CNN
+F 2 "Power_Integrations:TO-220" H 10300 1600 50  0001 C CNN
 F 3 "" H 9750 1600 60  0000 C CNN
 	1    9750 1600
@@
 U 1 1 56CF85BD
 P 3150 6700
-F 0 "U5" H 3150 6700 0   0001 C CNN
-F 1 "10-XX_B3F-10XX" H 3150 6700 0   0001 C CNN
+F 0 "U5" H 3150 6700 60  0001 C CNN
+F 1 "10-XX_B3F-10XX" H 3150 6700 60  0001 C CNN
 F 2 "switch-omron:B3F-10XX" H 3150 6700 60  0001 C CNN
 F 3 "" H 3150 6700 60  0000 C CNN

Commit message: progress
Parts:
- removed J1: audio-jack, audio-jack-lapantech:JACK_LAPAN, symbol audio-jack
- removed R4: 4k7, Resistors_SMD:R_0805, symbol R
- removed U5: 10-XX_B3F-10XX, switch-omron:B3F-10XX, symbol 10-XX_B3F-10XX
- renumbered J2 to J1
Connections:
- net ADC-BATT1: now also U1.14 (WKUP/USART2_CTS/ADC12_IN0/TIM2_CH1_ETR/PA0); no longer U1.15 (USART2_RTS/ADC12_IN1/TIM2_CH2/PA1)
- net ADC-BATT2: now also U1.15 (USART2_RTS/ADC12_IN1/TIM2_CH2/PA1); no longer U1.16 (USART2_TX/ADC12_IN2/TIM2_CH3/PA2)
- net ADC-DIM: now also U1.16 (USART2_TX/ADC12_IN2/TIM2_CH3/PA2); no longer U1.21 (SPI1_SCK/ADC12_IN5/PA5)
- net ADC-LAMP: now also U1.17 (USART2_RX/ADC12_IN3/TIM2_CH4/PA3); no longer U1.20 (SPI1_NSS/USART2_CK/ADC12_IN4/PA4)
- net ADC-USB: now also U1.20 (SPI1_NSS/USART2_CK/ADC12_IN4/PA4); no longer U1.17 (USART2_RX/ADC12_IN3/TIM2_CH4/PA3)
- net CON-LAMP: now also U1.33 (SPI2_NSS/I2C2_SMBA/USART3_CK/TIM1_BKIN/PB12); no longer U1.34 (SPI2_SCK/USART3_CTS/TIM1_CH1N/PB13)
- net CON-PV: now also U1.35 (SPI2_MISO/USART3_RTS/TIM1_CH2N/PB14); no longer U1.33 (SPI2_NSS/I2C2_SMBA/USART3_CK/TIM1_BKIN/PB12)
- net CON-USB: now also U1.34 (SPI2_SCK/USART3_CTS/TIM1_CH1N/PB13); no longer U1.35 (SPI2_MISO/USART3_RTS/TIM1_CH2N/PB14)
- net IND-PV: now also U1.21 (SPI1_SCK/ADC12_IN5/PA5); no longer U1.14 (WKUP/USART2_CTS/ADC12_IN0/TIM2_CH1_ETR/PA0)
- net BTN-USER: no longer names the net of U1.36 (SPI2_MOSI/TIM1_CH3N/PB15)
Other:
- moved on the sheet: D6, J1

Commit message: progress
Connections:
- net TX: now reaches P-COMM1.3 (P3), U1.42 (USART1_TX/TIM1_CH2/PA9)
- net RX: now reaches P-COMM1.4 (P4), U1.43 (USART1_RX/TIM1_CH3/PA10)
Changed lines of the file:
@@
 	0    1    1    0
 $EndComp
+Text Label 4950 2100 0    60   ~ 0
+TX
+Text Label 4900 2200 0    60   ~ 0
+RX
 $EndSCHEMATC

Commit message: standby mode
Connections:
- net ADC-BATT1: now also U1.21 (SPI1_SCK/ADC12_IN5/PA5); no longer U1.14 (WKUP/USART2_CTS/ADC12_IN0/TIM2_CH1_ETR/PA0)
- net IND-PV: now also U1.14 (WKUP/USART2_CTS/ADC12_IN0/TIM2_CH1_ETR/PA0); no longer U1.21 (SPI1_SCK/ADC12_IN5/PA5)
Changed lines of the file:
@@
 CON-USB
 Text Label 4900 1700 0    60   ~ 0
-IND-PV
+ADC-BATT1
 $Comp
 L GND #PWR013
@@
 IND-PV
 Text Label 4900 1200 0    60   ~ 0
-ADC-BATT1
+IND-PV
 $Comp
 L R R5

Commit message: progress
Parts:
- added R?: 4k7, Resistors_SMD:R_0805, symbol R
Connections:
- net GND: now also R?.2
- net IND-PV: now also R?.1
Changed lines of the file:
@@
 	6650 1300 6600 1300
 Wire Wire Line
-	6650 1500 6550 1500
-Text Label 6550 1500 0    60   ~ 0
-IND-PV
+	6350 1500 6650 1500
 Text Label 4900 1200 0    60   ~ 0
 IND-PV
@@
 Text Label 4900 2200 0    60   ~ 0
 RX
+$Comp
+L R R?
+U 1 1 56F3DD46
+P 6450 1650
+F 0 "R?" V 6530 1650 50  0000 C CNN
+F 1 "4k7" V 6450 1650 50  0000 C CNN
+F 2 "Resistors_SMD:R_0805" V 6380 1650 50  0001 C CNN
+F 3 "" H 6450 1650 50  0000 C CNN
+	1    6450 1650
+	1    0    0    -1
+$EndComp
+Connection ~ 6450 1500
+Text Label 6350 1500 0    60   ~ 0
+IND-PV
+$Comp
+L GND #PWR?
+U 1 1 56F3F6FF
+P 6450 1850
+F 0 "#PWR?" H 6450 1600 50  0001 C CNN
+F 1 "GND" H 6450 1700 50  0000 C CNN
+F 2 "" H 6450 1850 50  0000 C CNN
+F 3 "" H 6450 1850 50  0000 C CNN
+	1    6450 1850
+	1    0    0    -1
+$EndComp
+Wire Wire Line
+	6450 1800 6450 1850
 $EndSCHEMATC
